Commit message: vt0.1

File: src/rc_arm2_description/arm2.urdf (robot description, URDF)
Before this commit: robot arm2, 5 links, 4 joints
Links:
- added link tool0
Joints:
- added joint tool0_fixed: type fixed, parent l4, child tool0, origin xyz=0 0 0.0624 rpy=0 0 0

Commit message: vt1.0

File: src/rc_arm2_description/arm2.urdf (robot description, URDF)
Before this commit: robot arm2, 6 links, 5 joints
Joints:
- joint j1: limit lower=-3.14159 upper=3.14159 effort=10 velocity=1.0 -> lower=-3.14159 upper=3.14159 effort=10 velocity=3.0
- joint j2: limit lower=-3.14159 upper=3.14159 effort=10 velocity=1.0 -> lower=-3.14159 upper=3.14159 effort=10 velocity=3.0
- joint j3: limit lower=-3.14159 upper=3.14159 effort=10 velocity=1.0 -> lower=-3.14159 upper=3.14159 effort=10 velocity=3.0
- joint j4: limit lower=-3.14159 upper=3.14159 effort=10 velocity=1.0 -> lower=-3.14159 upper=3.14159 effort=10 velocity=3.0

Commit message: v3.7

File: src/rc_arm2_description/arm2.urdf (robot description, URDF)
Before this commit: robot arm2, 6 links, 5 joints
Joints:
- joint j1: limit lower=-3.14159 upper=3.14159 effort=10 velocity=3.0 -> lower=-3.14159 upper=3.14159 effort=10 velocity=12.0
- joint j2: limit lower=-3.14159 upper=3.14159 effort=10 velocity=3.0 -> lower=-3.14159 upper=3.14159 effort=10 velocity=12.0
- joint j3: limit lower=-3.14159 upper=3.14159 effort=10 velocity=3.0 -> lower=-3.14159 upper=3.14159 effort=10 velocity=12.0
- joint j4: limit lower=-3.14159 upper=3.14159 effort=10 velocity=3.0 -> lower=-3.14159 upper=3.14159 effort=10 velocity=12.0

Commit message: v3.9

File: src/rc_arm2_description/arm2.urdf (robot description, URDF)
Before this commit: robot arm2, 6 links, 5 joints
Joints:
- joint tool0_fixed: origin xyz=0 0 0.0624 rpy=0 0 0 -> xyz=0.01 -0.04 0.03 rpy=0 0 0

Commit message: mpvli0.1

File: src/rc_arm2_description/arm2.urdf (robot description, URDF)
Before this commit: robot arm2, 6 links, 5 joints
Joints:
- joint j1: limit lower=-3.14159 upper=3.14159 effort=10 velocity=12.0 -> lower=-1.865 upper=2.365 effort=10 velocity=12.0
- joint j2: limit lower=-3.14159 upper=3.14159 effort=10 velocity=12.0 -> lower=0.0 upper=1.85 effort=10 velocity=12.0
- joint j3: limit lower=-3.14159 upper=3.14159 effort=10 velocity=12.0 -> lower=0.0 upper=2.13861 effort=10 velocity=12.0
